Commit message: gazebo中加载机器人模型

File: chapt6/chapt6_ws/src/fishbot_description/urdf/fishbot/actuator/caster.urdf.xacro (robot description, xacro)
@@ -1,4 +1,5 @@
 <?xml version="1.0"?>
 <robot xmlns:xacro="http://www.ros.org/wiki/xacro">
+    <xacro:include filename="$(find fishbot_description)/urdf/fishbot/common_inertia.xacro" />
     <xacro:macro name="caster_xacro" params="caster_name xyz">
         <link name="${caster_name}_caster_link">
@@ -22,5 +23,12 @@
                 </material>
             </collision>
+            <xacro:sphere_inertia m="0.01" r="0.016" />
         </link>
+        <gazebo reference="${caster_name}_caster_link">
+            <mu1 value="0.0" />
+            <mu2 value="0.0" />
+            <kp value="1000000000.0" />
+            <kd value="1.0" />
+        </gazebo>
         <joint name="${caster_name}_caster_joint" type="fixed">
             <parent link="base_link" />

File: chapt6/chapt6_ws/src/fishbot_description/urdf/fishbot/actuator/wheel.urdf.xacro (robot description, xacro)
@@ -1,4 +1,5 @@
 <?xml version="1.0"?>
 <robot xmlns:xacro="http://www.ros.org/wiki/xacro">
+    <xacro:include filename="$(find fishbot_description)/urdf/fishbot/common_inertia.xacro" />
     <xacro:macro name="wheel_xacro" params="wheel_name xyz">
         <link name="${wheel_name}_wheel_link">
@@ -24,5 +25,18 @@
                 </material>
             </collision>
+            <xacro:cylinder_inertia m="0.1" h="0.04" r="0.032"/>
         </link>
+        <!--
+            mu1为切向摩擦系数
+            mu2为法向摩擦系数
+            kp表示接触的刚度系数
+            kd表示阻尼系数
+         -->
+        <gazebo reference="${wheel_name}_wheel_link">
+            <mu1 value="20.0" />
+            <mu2 value="20.0" />
+            <kp value="1000000000.0" />
+            <kd value="1.0" />
+        </gazebo>
         <joint name="${wheel_name}_wheel_joint" type="continuous">
         <!-- 轮子可以转，因此类型选择可转动的：continuous -->

File: chapt6/chapt6_ws/src/fishbot_description/urdf/fishbot/base.urdf.xacro (robot description, xacro)
@@ -1,4 +1,5 @@
 <?xml version="1.0"?>
 <robot xmlns:xacro="http://www.ros.org/wiki/xacro">
+    <xacro:include filename="$(find fishbot_description)/urdf/fishbot/common_inertia.xacro" />
     <xacro:macro name="base_xacro" params="length radius">
         <link name="base_footprint" />
@@ -33,4 +34,5 @@
                 </material>
             </collision>
+            <xacro:cylinder_inertia m="1.0" r="${radius}" h="${length}"/>
         </link>
     </xacro:macro>

File: chapt6/chapt6_ws/src/fishbot_description/urdf/fishbot/fishbot.urdf.xacro (robot description, xacro)
@@ -12,4 +12,6 @@
     <xacro:include filename="$(find fishbot_description)/urdf/fishbot/actuator/wheel.urdf.xacro" />
     <xacro:include filename="$(find fishbot_description)/urdf/fishbot/actuator/caster.urdf.xacro" />
+    <!-- Gazebo 插件 -->
+    <xacro:include filename="$(find fishbot_description)/urdf/fishbot/plugins/gazebo_control_plugin.xacro" />
     <!-- 调用宏 -->
     <xacro:base_xacro length="0.12" radius="0.1" />
@@ -24,3 +26,4 @@
     <xacro:caster_xacro caster_name="front" xyz="0.08 0.0 -0.076" />
     <xacro:caster_xacro caster_name="back" xyz="-0.08 0.0 -0.076" />
+    <xacro:gazebo_control_plugin />
 </robot>

File: chapt6/chapt6_ws/src/fishbot_description/urdf/fishbot/sensor/camera.urdf.xacro (robot description, xacro)
@@ -1,4 +1,5 @@
 <?xml version="1.0"?>
 <robot xmlns:xacro="http://www.ros.org/wiki/xacro">
+    <xacro:include filename="$(find fishbot_description)/urdf/fishbot/common_inertia.xacro" />
     <xacro:macro name="camera_xacro" params="xyz">
         <!-- ============相机模块================ -->
@@ -23,11 +24,6 @@
                 </material>
             </collision>
+            <xacro:box_inertia m="0.01" w="0.02" h="0.10" d="0.02" />
         </link>
-        <link name="camera_optical_link"></link>
-        <joint name="camera_optical_joint" type="fixed">
-            <parent link="camera_link" />
-            <child link="camera_optical_link" />
-            <origin xyz="0 0 0" rpy="${-pi/2} 0 ${-pi/2}" />
-        </joint>
         <joint name="camera_joint" type="fixed">
             <parent link="base_link" />

File: chapt6/chapt6_ws/src/fishbot_description/urdf/fishbot/sensor/imu.urdf.xacro (robot description, xacro)
@@ -1,4 +1,5 @@
 <?xml version="1.0"?>
 <robot xmlns:xacro="http://www.ros.org/wiki/xacro">
+    <xacro:include filename="$(find fishbot_description)/urdf/fishbot/common_inertia.xacro" />
     <xacro:macro name="imu_xacro" params="xyz">
         <!-- 机器人的imu部件，惯性测量传感器 -->
@@ -26,4 +27,5 @@
                 </material>
             </collision>
+            <xacro:box_inertia m="0.01" w="0.02" d="0.02" h="0.02"/>
         </link>
         <!-- 机器人的关节，用于组合机器人的部件 -->

File: chapt6/chapt6_ws/src/fishbot_description/urdf/fishbot/sensor/laser.urdf.xacro (robot description, xacro)
@@ -1,4 +1,5 @@
 <?xml version="1.0"?>
 <robot xmlns:xacro="http://www.ros.org/wiki/xacro">
+    <xacro:include filename="$(find fishbot_description)/urdf/fishbot/common_inertia.xacro" />
     <xacro:macro name="laser_xacro" params="xyz">
         <!-- ============雷达支撑杆================ -->
@@ -22,4 +23,5 @@
                 </material>
             </collision>
+            <xacro:cylinder_inertia m="0.01" r="0.01" h="0.10" />
         </link>
         <!-- 雷达支撑杆固定到base_link上 -->
@@ -49,4 +51,5 @@
                 </material>
             </collision>
+            <xacro:cylinder_inertia m="0.03" r="0.02" h="0.02" />
         </link>
         <!-- 雷达固定到雷达支撑杆上 -->
@@ -56,4 +59,10 @@
             <origin xyz="0 0 0.05" rpy="0.0 0.0 0.0"/>
         </joint>
+        <gazebo reference="laser_cylinder_link">
+            <material>Gazebo/Black</material>
+        </gazebo>
+        <gazebo reference="laser_link">
+            <material>Gazebo/Black</material>
+        </gazebo>
     </xacro:macro>
 </robot>
