Commit message: 激光雷达,imu,深度相机传感器仿真

File: chapt6/chapt6_ws/src/fishbot_description/urdf/fishbot/fishbot.urdf.xacro (robot description, xacro)
@@ -14,4 +14,5 @@
     <!-- Gazebo 插件 -->
     <xacro:include filename="$(find fishbot_description)/urdf/fishbot/plugins/gazebo_control_plugin.xacro" />
+    <xacro:include filename="$(find fishbot_description)/urdf/fishbot/plugins/gazebo_sensor_plugin.xacro" />
     <!-- 调用宏 -->
     <xacro:base_xacro length="0.12" radius="0.1" />
@@ -27,3 +28,4 @@
     <xacro:caster_xacro caster_name="back" xyz="-0.08 0.0 -0.076" />
     <xacro:gazebo_control_plugin />
+    <xacro:gazebo_sensor_plugin />
 </robot>

File: chapt6/chapt6_ws/src/fishbot_description/urdf/fishbot/sensor/camera.urdf.xacro (robot description, xacro)
@@ -26,4 +26,10 @@
             <xacro:box_inertia m="0.01" w="0.02" h="0.10" d="0.02" />
         </link>
+        <link name="camera_optical_link"></link>
+        <joint name="camera_optical_joint" type="fixed">
+            <parent link="camera_link" />
+            <child link="camera_optical_link" />
+            <origin xyz="0 0 0" rpy="${-pi/2} 0 ${-pi/2}" />
+        </joint>
         <joint name="camera_joint" type="fixed">
             <parent link="base_link" />
